File: hardware/esp8266-dev.brd (EAGLE design)
At the start: 48.3 x 48.3 mm, 32 parts, among them CON1 USBB-SOCKET, IC2 3V3

Commit message: Cleaned up schematic
Parts:
- removed U$1: OSHW-LOGOS, SparkFun:OSHW-LOGO-S
Changed lines of the file:
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@@
 </element>
 <element name="SW1" library="p.peter-passives" package="SWITCH-GENERIC-4_PIN" value="" x="43.18" y="45.72" smashed="yes" rot="R90"/>
-<element name="U$1" library="SparkFun" package="OSHW-LOGO-S" value="OSHW-LOGOS" x="43.18" y="45.72"/>
 <element name="UC" library="SparkFun" package="DIP08" value="ATTINY85" x="33.02" y="7.62" smashed="yes" rot="R270">
 <attribute name="VALUE" x="34.29" y="7.62" size="1.27" layer="27" font="vector" ratio="12" rot="R270" align="center"/>
