File: hardware/esp8266-dev-ftdi.sch (EAGLE design)
At the start: 52 parts, among them CON1 USBMICRO-NO_CENTER-LONG_PADS

Commit message: board outline and orga
Parts:
- removed SW4: (no value), p.peter-passives:SWITCH-DEFAULT_OFF-2PIN
- added SW-RESET: (no value), p.peter-passives:SWITCH-DEFAULT_OFF-2PIN
Connections:
- net GND: now also SW-RESET.P$1; no longer SW2.P$1
- net N$20: now also SW2.P$1; no longer SW3.P$1
- net N$21: now also SW3.P$1; no longer SW4.P$1
- net RESET: now also SW-RESET.P$2; no longer SW2.P$2
- net RX: now also SW3.P$2; no longer SW4.P$2
- net TX: now also SW2.P$2; no longer SW3.P$2
Other:
- moved on the sheet: SW2, SW3
Changed lines of the file:
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@@
 <part name="GND21" library="supply1" deviceset="GND" device=""/>
 <part name="F1" library="p.peter-regulators" deviceset="FUSE" device="0805" value="500mA"/>
+<part name="SW-RESET" library="p.peter-passives" deviceset="SWITCH-DEFAULT_OFF" device="-2PIN"/>
 <part name="SW2" library="p.peter-passives" deviceset="SWITCH-DEFAULT_OFF" device="-2PIN"/>
 <part name="SW3" library="p.peter-passives" deviceset="SWITCH-DEFAULT_OFF" device="-2PIN"/>
-<part name="SW4" library="p.peter-passives" deviceset="SWITCH-DEFAULT_OFF" device="-2PIN"/>
 <part name="GND22" library="supply1" deviceset="GND" device=""/>
 <part name="R9" library="p.peter-rcl" deviceset="R-EU_" device="R0603" value="2k"/>
@@
 <attribute name="VALUE" x="134.62" y="58.42" size="1.778" layer="96" ratio="12" align="center"/>
 </instance>
-<instance part="SW2" gate="S$1" x="43.18" y="-38.1"/>
-<instance part="SW3" gate="S$1" x="38.1" y="-71.12"/>
-<instance part="SW4" gate="S$1" x="38.1" y="-78.74"/>
+<instance part="SW-RESET" gate="S$1" x="43.18" y="-38.1"/>
+<instance part="SW2" gate="S$1" x="38.1" y="-71.12"/>
+<instance part="SW3" gate="S$1" x="38.1" y="-78.74"/>
 <instance part="GND22" gate="1" x="22.86" y="-45.72"/>
 <instance part="R9" gate="G$1" x="25.4" y="-71.12"/>
@@
 </segment>
 <segment>
-<pinref part="SW2" gate="S$1" pin="P$1"/>
+<pinref part="SW-RESET" gate="S$1" pin="P$1"/>
 <wire x1="38.1" y1="-38.1" x2="22.86" y2="-38.1" width="0.1524" layer="91"/>
 <wire x1="22.86" y1="-38.1" x2="22.86" y2="-43.18" width="0.1524" layer="91"/>
@@
 <wire x1="58.42" y1="-71.12" x2="58.42" y2="-63.5" width="0.1524" layer="91"/>
 <label x="58.42" y="-63.5" size="1.27" layer="95" rot="R90" xref="yes"/>
-<pinref part="SW3" gate="S$1" pin="P$2"/>
+<pinref part="SW2" gate="S$1" pin="P$2"/>
 <wire x1="43.18" y1="-71.12" x2="58.42" y2="-71.12" width="0.1524" layer="91"/>
 <junction x="58.42" y="-71.12"/>
@@
 <wire x1="53.34" y1="-78.74" x2="53.34" y2="-63.5" width="0.1524" layer="91"/>
 <label x="53.34" y="-63.5" size="1.27" layer="95" rot="R90" xref="yes"/>
-<pinref part="SW4" gate="S$1" pin="P$2"/>
+<pinref part="SW3" gate="S$1" pin="P$2"/>
 <wire x1="43.18" y1="-78.74" x2="53.34" y2="-78.74" width="0.1524" layer="91"/>
 <junction x="53.34" y="-78.74"/>
@@
 <wire x1="55.88" y1="-40.64" x2="55.88" y2="-38.1" width="0.1524" layer="91"/>
 <junction x="55.88" y="-38.1"/>
-<pinref part="SW2" gate="S$1" pin="P$2"/>
+<pinref part="SW-RESET" gate="S$1" pin="P$2"/>
 <wire x1="55.88" y1="-38.1" x2="48.26" y2="-38.1" width="0.1524" layer="91"/>
 </segment>
@@
 <segment>
 <pinref part="R9" gate="G$1" pin="2"/>
+<pinref part="SW2" gate="S$1" pin="P$1"/>
+<wire x1="30.48" y1="-71.12" x2="33.02" y2="-71.12" width="0.1524" layer="91"/>
+</segment>
+</net>
+<net name="N$21" class="0">
+<segment>
 <pinref part="SW3" gate="S$1" pin="P$1"/>
-<wire x1="30.48" y1="-71.12" x2="33.02" y2="-71.12" width="0.1524" layer="91"/>
-</segment>
-</net>
-<net name="N$21" class="0">
-<segment>
-<pinref part="SW4" gate="S$1" pin="P$1"/>
 <pinref part="R10" gate="G$1" pin="2"/>
 <wire x1="30.48" y1="-78.74" x2="33.02" y2="-78.74" width="0.1524" layer="91"/>

Commit message: LED power
Parts:
- removed TP1, TP10, TP11, TP2, TP3, TP4, TP5, TP6, TP7, TP8, TP9: TPSQTP15R, testpad:TPSQTP15R
- C2, C3, C4, C5, C6: device p.peter-rcl:C-EUC0603 -> p.peter-rcl:C-EUC0805
- R1, R10, R11, R2, R3, R4, R5, R6, R7, R8, R9: device p.peter-rcl:R-EU_R0603 -> p.peter-rcl:R-EU_R0805
Connections:
- net +3V3: no longer TP10.TP
- net +5V: no longer TP9.TP
- net /PWREN: no longer TP7.TP
- net /SLEEP: no longer TP6.TP
- net CTS: no longer TP2.TP
- net GND: no longer TP11.TP
- net RESET: no longer TP5.TP
- net RTS: no longer TP1.TP
- net RX: no longer TP3.TP
- net TX: no longer TP4.TP
- net VCCIO: no longer TP8.TP
Other:
- moved on the sheet: L1

Commit message: Everything routed
Parts:
- JP1: device pinhead:PINHD-2X5 -> p.peter-connectors:GENERIC-2X5
Connections:
- net +5V: now also JP1.10; no longer JP1.1
- net /PWREN: now also U$1.CBUS2; no longer U$1.CBUS3
- net /SLEEP: now also U$1.CBUS3; no longer U$1.CBUS0
- net GND: now also JP1.9; no longer JP1.4
- net IO16: now also JP1.1; no longer JP1.10
- net N$13: now also U$1.CBUS0; no longer U$1.CBUS2
- net RESET: now also JP1.2; no longer JP1.9
- net RX: now also JP1.4; no longer JP1.5
- net TX: now also JP1.5; no longer JP1.7
- net VCCIO: now also JP1.7; no longer JP1.2
Other:
- moved on the sheet: LED-RX, LED-TX, R3, R4
Changed lines of the file:
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@@
 <part name="SJ2" library="jumper" deviceset="SJ2W" device=""/>
 <part name="P+12" library="supply1" deviceset="+5V" device=""/>
-<part name="JP1" library="pinhead" deviceset="PINHD-2X5" device=""/>
+<part name="JP1" library="p.peter-connectors" deviceset="GENERIC-2X5" device=""/>
 <part name="P+13" library="supply1" deviceset="+5V" device=""/>
 <part name="+3V5" library="supply1" deviceset="+3V3" device=""/>
@@
 <instance part="GND6" gate="1" x="2.54" y="27.94"/>
 <instance part="GND7" gate="1" x="12.7" y="27.94"/>
-<instance part="LED-TX" gate="G$1" x="88.9" y="10.16" rot="R270"/>
-<instance part="LED-RX" gate="G$1" x="96.52" y="12.7" rot="R270"/>
-<instance part="R3" gate="G$1" x="88.9" y="20.32" rot="R90"/>
-<instance part="R4" gate="G$1" x="96.52" y="22.86" rot="R90"/>
-<instance part="GND8" gate="1" x="88.9" y="0"/>
-<instance part="GND9" gate="1" x="96.52" y="0"/>
+<instance part="LED-TX" gate="G$1" x="96.52" y="10.16" rot="R270"/>
+<instance part="LED-RX" gate="G$1" x="88.9" y="10.16" rot="R270"/>
+<instance part="R3" gate="G$1" x="96.52" y="20.32" rot="R90"/>
+<instance part="R4" gate="G$1" x="88.9" y="20.32" rot="R90"/>
+<instance part="GND8" gate="1" x="96.52" y="0"/>
+<instance part="GND9" gate="1" x="88.9" y="0"/>
 <instance part="LED1" gate="G$1" x="223.52" y="-30.48" rot="R270"/>
 <instance part="+3V2" gate="G$1" x="210.82" y="-25.4"/>
@@
 <instance part="SJ2" gate="G$1" x="25.4" y="48.26" rot="R180"/>
 <instance part="P+12" gate="1" x="25.4" y="38.1" rot="R180"/>
-<instance part="JP1" gate="A" x="231.14" y="45.72"/>
+<instance part="JP1" gate="G$1" x="231.14" y="45.72"/>
 <instance part="P+13" gate="1" x="223.52" y="58.42"/>
 <instance part="+3V5" gate="G$1" x="215.9" y="58.42"/>
@@
 <pinref part="LED-TX" gate="G$1" pin="C"/>
 <pinref part="GND8" gate="1" pin="GND"/>
-<wire x1="88.9" y1="2.54" x2="88.9" y2="5.08" width="0.1524" layer="91"/>
+<wire x1="96.52" y1="2.54" x2="96.52" y2="5.08" width="0.1524" layer="91"/>
 </segment>
 <segment>
 <pinref part="LED-RX" gate="G$1" pin="C"/>
 <pinref part="GND9" gate="1" pin="GND"/>
-<wire x1="96.52" y1="2.54" x2="96.52" y2="7.62" width="0.1524" layer="91"/>
+<wire x1="88.9" y1="2.54" x2="88.9" y2="5.08" width="0.1524" layer="91"/>
 </segment>
 <segment>
@@
 </segment>
 <segment>
-<pinref part="JP1" gate="A" pin="4"/>
+<pinref part="JP1" gate="G$1" pin="9"/>
 <pinref part="GND24" gate="1" pin="GND"/>
-<wire x1="236.22" y1="48.26" x2="254" y2="48.26" width="0.1524" layer="91"/>
+<wire x1="226.06" y1="40.64" x2="254" y2="48.26" width="0.1524" layer="91"/>
 <wire x1="254" y1="48.26" x2="254" y2="43.18" width="0.1524" layer="91"/>
 </segment>
@@
 </segment>
 <segment>
-<pinref part="JP1" gate="A" pin="1"/>
+<pinref part="JP1" gate="G$1" pin="10"/>
 <pinref part="P+13" gate="1" pin="+5V"/>
-<wire x1="228.6" y1="50.8" x2="223.52" y2="50.8" width="0.1524" layer="91"/>
+<wire x1="233.68" y1="40.64" x2="223.52" y2="50.8" width="0.1524" layer="91"/>
 <wire x1="223.52" y1="50.8" x2="223.52" y2="55.88" width="0.1524" layer="91"/>
 </segment>
@@
 </segment>
 <segment>
-<pinref part="JP1" gate="A" pin="7"/>
-<wire x1="228.6" y1="43.18" x2="223.52" y2="43.18" width="0.1524" layer="91"/>
+<pinref part="JP1" gate="G$1" pin="5"/>
+<wire x1="226.06" y1="45.72" x2="223.52" y2="43.18" width="0.1524" layer="91"/>
 <label x="223.52" y="43.18" size="1.27" layer="95" rot="R180" xref="yes"/>
 </segment>
@@
 </segment>
 <segment>
-<pinref part="JP1" gate="A" pin="5"/>
-<wire x1="228.6" y1="45.72" x2="223.52" y2="45.72" width="0.1524" layer="91"/>
+<pinref part="JP1" gate="G$1" pin="4"/>
+<wire x1="233.68" y1="48.26" x2="223.52" y2="45.72" width="0.1524" layer="91"/>
 <label x="223.52" y="45.72" size="1.27" layer="95" rot="R180" xref="yes"/>
 </segment>
@@
 <net name="/SLEEP" class="0">
 <segment>
-<pinref part="U$1" gate="G$1" pin="CBUS0"/>
-<wire x1="73.66" y1="33.02" x2="76.2" y2="33.02" width="0.1524" layer="91"/>
-<label x="76.2" y="33.02" size="1.27" layer="95" xref="yes"/>
+<pinref part="U$1" gate="G$1" pin="CBUS3"/>
+<wire x1="73.66" y1="25.4" x2="76.2" y2="25.4" width="0.1524" layer="91"/>
+<label x="76.2" y="25.4" size="1.27" layer="95" xref="yes"/>
 </segment>
 <segment>
@@
 <net name="/PWREN" class="0">
 <segment>
-<pinref part="U$1" gate="G$1" pin="CBUS3"/>
-<wire x1="73.66" y1="25.4" x2="76.2" y2="25.4" width="0.1524" layer="91"/>
-<label x="76.2" y="25.4" size="1.27" layer="95" xref="yes"/>
+<pinref part="U$1" gate="G$1" pin="CBUS2"/>
+<wire x1="73.66" y1="27.94" x2="76.2" y2="27.94" width="0.1524" layer="91"/>
+<label x="76.2" y="27.94" size="1.27" layer="95" xref="yes"/>
 </segment>
 <segment>
@@
 <net name="N$13" class="0">
 <segment>
-<pinref part="U$1" gate="G$1" pin="CBUS2"/>
-<wire x1="73.66" y1="27.94" x2="76.2" y2="27.94" width="0.1524" layer="91"/>
+<pinref part="U$1" gate="G$1" pin="CBUS0"/>
+<wire x1="73.66" y1="33.02" x2="83.82" y2="33.02" width="0.1524" layer="91"/>
 <pinref part="R3" gate="G$1" pin="2"/>
-<wire x1="76.2" y1="27.94" x2="88.9" y2="27.94" width="0.1524" layer="91"/>
-<wire x1="88.9" y1="27.94" x2="88.9" y2="25.4" width="0.1524" layer="91"/>
+<wire x1="83.82" y1="33.02" x2="96.52" y2="33.02" width="0.1524" layer="91"/>
+<wire x1="96.52" y1="33.02" x2="96.52" y2="25.4" width="0.1524" layer="91"/>
 </segment>
 </net>
@@
 <segment>
 <pinref part="U$1" gate="G$1" pin="CBUS1"/>
-<wire x1="73.66" y1="30.48" x2="76.2" y2="30.48" width="0.1524" layer="91"/>
-<wire x1="76.2" y1="30.48" x2="96.52" y2="30.48" width="0.1524" layer="91"/>
-<wire x1="96.52" y1="30.48" x2="96.52" y2="27.94" width="0.1524" layer="91"/>
+<wire x1="73.66" y1="30.48" x2="88.9" y2="30.48" width="0.1524" layer="91"/>
+<wire x1="88.9" y1="30.48" x2="88.9" y2="25.4" width="0.1524" layer="91"/>
 <pinref part="R4" gate="G$1" pin="2"/>
 </segment>
@@
 <pinref part="R3" gate="G$1" pin="1"/>
 <pinref part="LED-TX" gate="G$1" pin="A"/>
-<wire x1="88.9" y1="12.7" x2="88.9" y2="15.24" width="0.1524" layer="91"/>
+<wire x1="96.52" y1="12.7" x2="96.52" y2="15.24" width="0.1524" layer="91"/>
 </segment>
 </net>
@@
 <pinref part="R4" gate="G$1" pin="1"/>
 <pinref part="LED-RX" gate="G$1" pin="A"/>
-<wire x1="96.52" y1="15.24" x2="96.52" y2="17.78" width="0.1524" layer="91"/>
+<wire x1="88.9" y1="12.7" x2="88.9" y2="15.24" width="0.1524" layer="91"/>
 </segment>
 </net>
@@
 </segment>
 <segment>
-<pinref part="JP1" gate="A" pin="3"/>
+<pinref part="JP1" gate="G$1" pin="3"/>
 <pinref part="+3V5" gate="G$1" pin="+3V3"/>
-<wire x1="228.6" y1="48.26" x2="215.9" y2="48.26" width="0.1524" layer="91"/>
+<wire x1="226.06" y1="48.26" x2="215.9" y2="48.26" width="0.1524" layer="91"/>
 <wire x1="215.9" y1="48.26" x2="215.9" y2="55.88" width="0.1524" layer="91"/>
 </segment>
@@
 </segment>
 <segment>
-<pinref part="JP1" gate="A" pin="9"/>
-<wire x1="228.6" y1="40.64" x2="223.52" y2="40.64" width="0.1524" layer="91"/>
+<pinref part="JP1" gate="G$1" pin="2"/>
+<wire x1="233.68" y1="50.8" x2="223.52" y2="40.64" width="0.1524" layer="91"/>
 <label x="223.52" y="40.64" size="1.27" layer="95" rot="R180" xref="yes"/>
 </segment>
@@
 </segment>
 <segment>
-<pinref part="JP1" gate="A" pin="8"/>
-<wire x1="236.22" y1="43.18" x2="241.3" y2="43.18" width="0.1524" layer="91"/>
+<pinref part="JP1" gate="G$1" pin="8"/>
+<wire x1="233.68" y1="43.18" x2="241.3" y2="43.18" width="0.1524" layer="91"/>
 <label x="241.3" y="43.18" size="1.27" layer="95" xref="yes"/>
 </segment>
@@
 </segment>
 <segment>
-<pinref part="JP1" gate="A" pin="10"/>
-<wire x1="236.22" y1="40.64" x2="241.3" y2="40.64" width="0.1524" layer="91"/>
+<pinref part="JP1" gate="G$1" pin="1"/>
+<wire x1="226.06" y1="50.8" x2="241.3" y2="40.64" width="0.1524" layer="91"/>
 <label x="241.3" y="40.64" size="1.27" layer="95" xref="yes"/>
 </segment>
@@
 </segment>
 <segment>
-<pinref part="JP1" gate="A" pin="6"/>
-<wire x1="236.22" y1="45.72" x2="241.3" y2="45.72" width="0.1524" layer="91"/>
+<pinref part="JP1" gate="G$1" pin="6"/>
+<wire x1="233.68" y1="45.72" x2="241.3" y2="45.72" width="0.1524" layer="91"/>
 <label x="241.3" y="45.72" size="1.27" layer="95" xref="yes"/>
 </segment>
@@
 </segment>
 <segment>
-<pinref part="JP1" gate="A" pin="2"/>
-<wire x1="236.22" y1="50.8" x2="243.84" y2="50.8" width="0.1524" layer="91"/>
+<pinref part="JP1" gate="G$1" pin="7"/>
+<wire x1="226.06" y1="43.18" x2="243.84" y2="50.8" width="0.1524" layer="91"/>
 <wire x1="243.84" y1="50.8" x2="243.84" y2="53.34" width="0.1524" layer="91"/>
 <label x="243.84" y="53.34" size="1.27" layer="95" rot="R90" xref="yes"/>

Commit message: Layout done
Parts:
- removed SW3: (no value), p.peter-passives:SWITCH-DEFAULT_OFF-2PIN
- added FLASH: (no value), p.peter-passives:SWITCH-DEFAULT_OFF-DEFAULT
- added SLEEP: (no value), jumper:SJ
- RF1: device p.peter-periphery:ESP2866-ESP-01THT-NOSILK -> p.peter-periphery:ESP2866-ESP-01THT
- SW1: device p.peter-passives:SWITCH-DEFAULT_OFF-DEFAULT -> p.peter-passives:SWITCH-DEFAULT_OFF-2PIN
- renumbered SW-RESET to RESET, U$1 to FT230
Connections:
- new net N$10: SLEEP.2, U$2.DTR
- net /SLEEP: now also SLEEP.1; no longer U$2.DTR
- net GND: now also FLASH.P$2; no longer SW1.P$2
- net N$11: now also FLASH.P$1; no longer SW1.P$1
- net N$21: now also SW1.P$1; no longer SW3.P$1
- net RX: now also SW1.P$2; no longer SW3.P$2
Other:
- moved on the sheet: SW1

Commit message: MVP
Parts:
- U$2: value UART-6_PIN -> UART-6_PINGENERIC; device p.peter-connectors:UART-6_PIN -> p.peter-connectors:UART-6_PINGENERIC
Changed lines of the file:
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@@
 <part name="R7" library="p.peter-rcl" deviceset="R-EU_" device="R0805" value="10k"/>
 <part name="GND13" library="supply1" deviceset="GND" device=""/>
-<part name="U$2" library="p.peter-connectors" deviceset="UART-6_PIN" device=""/>
+<part name="U$2" library="p.peter-connectors" deviceset="UART-6_PIN" device="GENERIC"/>
 <part name="GND15" library="supply1" deviceset="GND" device=""/>
 <part name="+3V4" library="supply1" deviceset="+3V3" device=""/>

Commit message: added test pads
Parts:
- added 3V3, 5V, CTS, GND, PEN, RES, RTS, RX, SLE, TX, VCC: TPSQTP15R, testpad:TPSQTP15R
Connections:
- net +3V3: now also 3V3.TP
- net +5V: now also 5V.TP
- net /PWREN: now also PEN.TP
- net /SLEEP: now also SLE.TP
- net CTS: now also CTS.TP
- net GND: now also GND.TP
- net RESET: now also RES.TP
- net RTS: now also RTS.TP
- net RX: now also RX.TP
- net TX: now also TX.TP
- net VCCIO: now also VCC.TP
Changed lines of the file:
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@@
 <part name="GND14" library="supply1" deviceset="GND" device=""/>
 <part name="SLEEP" library="jumper" deviceset="SJ" device=""/>
+<part name="RTS" library="testpad" deviceset="TPSQ" device="TP15R"/>
+<part name="CTS" library="testpad" deviceset="TPSQ" device="TP15R"/>
+<part name="RX" library="testpad" deviceset="TPSQ" device="TP15R"/>
+<part name="TX" library="testpad" deviceset="TPSQ" device="TP15R"/>
+<part name="RES" library="testpad" deviceset="TPSQ" device="TP15R"/>
+<part name="SLE" library="testpad" deviceset="TPSQ" device="TP15R"/>
+<part name="PEN" library="testpad" deviceset="TPSQ" device="TP15R"/>
+<part name="VCC" library="testpad" deviceset="TPSQ" device="TP15R"/>
+<part name="5V" library="testpad" deviceset="TPSQ" device="TP15R"/>
+<part name="3V3" library="testpad" deviceset="TPSQ" device="TP15R"/>
+<part name="GND" library="testpad" deviceset="TPSQ" device="TP15R"/>
 </parts>
 <sheets>
@@
 <instance part="GND14" gate="1" x="78.74" y="78.74" rot="R180"/>
 <instance part="SLEEP" gate="1" x="154.94" y="20.32"/>
+<instance part="RTS" gate="G$1" x="25.4" y="71.12"/>
+<instance part="CTS" gate="G$1" x="30.48" y="71.12"/>
+<instance part="RX" gate="G$1" x="35.56" y="71.12"/>
+<instance part="TX" gate="G$1" x="40.64" y="71.12"/>
+<instance part="RES" gate="G$1" x="45.72" y="71.12"/>
+<instance part="SLE" gate="G$1" x="50.8" y="71.12"/>
+<instance part="PEN" gate="G$1" x="55.88" y="71.12"/>
+<instance part="VCC" gate="G$1" x="63.5" y="71.12"/>
+<instance part="5V" gate="G$1" x="68.58" y="71.12"/>
+<instance part="3V3" gate="G$1" x="73.66" y="71.12"/>
+<instance part="GND" gate="G$1" x="78.74" y="71.12"/>
 </instances>
 <busses>
@@
 <pinref part="GND14" gate="1" pin="GND"/>
 <wire x1="78.74" y1="76.2" x2="78.74" y2="73.66" width="0.1524" layer="91"/>
+<pinref part="GND" gate="G$1" pin="TP"/>
 </segment>
 </net>
@@
 <pinref part="P+6" gate="1" pin="+5V"/>
 <wire x1="68.58" y1="76.2" x2="68.58" y2="73.66" width="0.1524" layer="91"/>
+<pinref part="5V" gate="G$1" pin="TP"/>
 </segment>
 </net>
@@
 <wire x1="40.64" y1="73.66" x2="40.64" y2="76.2" width="0.1524" layer="91"/>
 <label x="40.64" y="76.2" size="1.27" layer="95" rot="R90" xref="yes"/>
+<pinref part="TX" gate="G$1" pin="TP"/>
 </segment>
 </net>
@@
 <wire x1="35.56" y1="73.66" x2="35.56" y2="76.2" width="0.1524" layer="91"/>
 <label x="35.56" y="76.2" size="1.27" layer="95" rot="R90" xref="yes"/>
+<pinref part="RX" gate="G$1" pin="TP"/>
 </segment>
 </net>
@@
 <wire x1="50.8" y1="73.66" x2="50.8" y2="76.2" width="0.1524" layer="91"/>
 <label x="50.8" y="76.2" size="1.27" layer="95" rot="R90" xref="yes"/>
+<pinref part="SLE" gate="G$1" pin="TP"/>
 </segment>
 </net>
@@
 <wire x1="25.4" y1="73.66" x2="25.4" y2="76.2" width="0.1524" layer="91"/>
 <label x="25.4" y="76.2" size="1.27" layer="95" rot="R90" xref="yes"/>
+<pinref part="RTS" gate="G$1" pin="TP"/>
 </segment>
 </net>
@@
 <wire x1="30.48" y1="73.66" x2="30.48" y2="76.2" width="0.1524" layer="91"/>
 <label x="30.48" y="76.2" size="1.27" layer="95" rot="R90" xref="yes"/>
+<pinref part="CTS" gate="G$1" pin="TP"/>
 </segment>
 </net>
@@
 <wire x1="55.88" y1="73.66" x2="55.88" y2="76.2" width="0.1524" layer="91"/>
 <label x="55.88" y="76.2" size="1.27" layer="95" rot="R90" xref="yes"/>
+<pinref part="PEN" gate="G$1" pin="TP"/>
 </segment>
 </net>
@@
 <pinref part="+3V6" gate="G$1" pin="+3V3"/>
 <wire x1="73.66" y1="76.2" x2="73.66" y2="73.66" width="0.1524" layer="91"/>
+<pinref part="3V3" gate="G$1" pin="TP"/>
 </segment>
 </net>
@@
 <wire x1="45.72" y1="73.66" x2="45.72" y2="76.2" width="0.1524" layer="91"/>
 <label x="45.72" y="76.2" size="1.27" layer="95" rot="R90" xref="yes"/>
+<pinref part="RES" gate="G$1" pin="TP"/>
 </segment>
 </net>
@@
 <wire x1="63.5" y1="73.66" x2="63.5" y2="76.2" width="0.1524" layer="91"/>
 <label x="63.5" y="76.2" size="1.27" layer="95" rot="R90" xref="yes"/>
-</segment>
-</net>
+<pinref part="VCC" gate="G$1" pin="TP"/>
+</segment>
+</net>

Commit message: minor cleanup
Other:
- note removed: "TODO: - Footprints for 2mm V12, Breakoutboard - Prototype area with - Hooks for rubber band - Hole for lanyard"
Changed lines of the file:
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@@
 <wire x1="134.62" y1="-88.9" x2="134.62" y2="-15.24" width="0.4064" layer="97" style="shortdash"/>
 <wire x1="134.62" y1="-15.24" x2="2.54" y2="-15.24" width="0.4064" layer="97" style="shortdash"/>
-<text x="-25.4" y="-17.78" size="3.81" layer="97" ratio="15" align="top-left">ESP 8266
+<text x="104.14" y="-17.78" size="3.81" layer="97" ratio="15" align="top-left">ESP 8266
 Interface</text>
 <text x="144.78" y="-17.78" size="3.81" layer="97" ratio="15" align="top-left">Power
@@
 v0.1 (8e144a9ffe)
 </text>
-<text x="180.34" y="-7.62" size="2.54" layer="97" ratio="12">TODO:
-- Footprints for 2mm V12, Breakoutboard
-- Prototype area with
-- Hooks for rubber band
-- Hole for lanyard
-</text>
 </plain>
